Commit message: kinetic - remove collision box that may contribute to vibrations in simulation

File: kinova_description/urdf/j2n4s300_standalone.xacro (robot description, xacro)
@@ -23,10 +23,10 @@
     <!--<material name="Black" /> -->
     </visual>
-    <collision>
+    <!--collision>
       <origin xyz="0 0 0" rpy="0 0 0" />
       <geometry>
         <box size = "0.01 0.01 0.01"/>
       </geometry>
-    </collision>
+    </collision-->
   </link>
   <!-- for gazebo -->

File: kinova_description/urdf/j2n6s200_standalone.xacro (robot description, xacro)
@@ -23,10 +23,10 @@
     <!--<material name="Black" /> -->
     </visual>
-    <collision>
+		<!--collision>
       <origin xyz="0 0 0" rpy="0 0 0" />
       <geometry>
         <box size = "0.01 0.01 0.01"/>
       </geometry>
-    </collision>
+    </collision-->
   </link>
   <!-- for gazebo -->

File: kinova_description/urdf/j2n6s300_standalone.xacro (robot description, xacro)
@@ -23,10 +23,10 @@
     <!--<material name="Black" /> -->
     </visual>
-    <collision>
+		<!--collision>
       <origin xyz="0 0 0" rpy="0 0 0" />
       <geometry>
         <box size = "0.01 0.01 0.01"/>
       </geometry>
-    </collision>
+    </collision-->
   </link>
   <!-- for gazebo -->

File: kinova_description/urdf/j2n7s300_standalone.xacro (robot description, xacro)
@@ -23,10 +23,10 @@
     <!--<material name="Black" /> -->
     </visual>
-    <collision>
+		<!--collision>
       <origin xyz="0 0 0" rpy="0 0 0" />
       <geometry>
         <box size = "0.01 0.01 0.01"/>
       </geometry>
-    </collision>
+    </collision-->
   </link>
   <!-- for gazebo -->

File: kinova_description/urdf/j2s6s300_standalone.xacro (robot description, xacro)
@@ -23,10 +23,10 @@
     <!--<material name="Black" /> -->
     </visual>
-    <collision>
+		<!--collision>
       <origin xyz="0 0 0" rpy="0 0 0" />
       <geometry>
         <box size = "0.01 0.01 0.01"/>
       </geometry>
-    </collision>
+    </collision-->
   </link>
   <!-- for gazebo -->

File: kinova_description/urdf/j2s7s300_standalone.xacro (robot description, xacro)
@@ -23,10 +23,10 @@
     <!--<material name="Black" /> -->
     </visual>
-    <collision>
+		<!--collision>
       <origin xyz="0 0 0" rpy="0 0 0" />
       <geometry>
         <box size = "0.01 0.01 0.01"/>
       </geometry>
-    </collision>
+    </collision-->
   </link>
   <!-- for gazebo -->

File: kinova_description/urdf/m1n6s300_standalone.xacro (robot description, xacro)
@@ -23,10 +23,10 @@
     <!--<material name="Black" /> -->
     </visual>
-    <collision>
+    <!--collision>
       <origin xyz="0 0 0" rpy="0 0 0" />
       <geometry>
         <box size = "0.01 0.01 0.01"/>
       </geometry>
-    </collision>
+    </collision-->
   </link>
   <!-- for gazebo -->
