Commit message: kinetic - add color to gazebo model; use implicit damper modeling; mimic joint for finger tip for RViz; use _driver namespace for controls

File: kinova_description/urdf/kinova_common.xacro (robot description, xacro)
@@ -26,7 +26,7 @@
                 </material>
             </visual>
-	    <!-- Adding ring to the model -->
-	         <xacro:if value="${use_ring_mesh}">
-	           <visual>
+           <!-- Adding ring to the model -->
+           <xacro:if value="${use_ring_mesh}">
+             <visual>
                 <geometry>
                     <mesh
@@ -34,5 +34,5 @@
                 </geometry>
              </visual>
-	    </xacro:if>
+           </xacro:if>
             <collision>
                 <geometry>
@@ -41,6 +41,16 @@
                 </geometry>
             </collision>
-						<xacro:kinova_inertial mesh_no="${mesh_no}"/>
-      </link>
+            <xacro:kinova_inertial mesh_no="${mesh_no}"/>
+            <gazebo reference="[links in contact]">
+              <kp>1000000.0</kp>
+              <kd>1.0</kd>
+              <mu1>1.0</mu1>
+              <mu2>1.0</mu2>
+              <minDepth>0.001</minDepth>
+            </gazebo>
+        </link>
+      <gazebo reference="${link_name}">
+          <material>Gazebo/DarkGrey</material>
+      </gazebo>
     </xacro:macro>
   <xacro:macro name="kinova_armjoint" params="joint_name type parent child joint_axis_xyz joint_origin_xyz joint_origin_rpy joint_lower_limit joint_upper_limit fixed:=false">
@@ -49,9 +59,12 @@
         <child link="${child}"/>
         <axis xyz="${joint_axis_xyz}"/>
-        <limit effort="2000" velocity="1" lower="${joint_lower_limit}" upper="${joint_upper_limit}"/>
+        <limit effort="60" velocity="6.28" lower="${joint_lower_limit}" upper="${joint_upper_limit}"/>
         <origin xyz="${joint_origin_xyz}" rpy="${joint_origin_rpy}"/>
-        <dynamics damping="0.0" friction="0.0"/>
+        <dynamics damping="1.7" friction="0.0"/>
      </joint>
    <xacro:unless value="${fixed}">
+     <gazebo reference="${joint_name}">
+        <implicitSpringDamper>1</implicitSpringDamper>
+     </gazebo>
      <transmission name="${joint_name}_trans">
         <type>transmission_interface/SimpleTransmission</type>
@@ -64,5 +77,5 @@
         </actuator>
      </transmission>
-     </xacro:unless>
+   </xacro:unless>
   </xacro:macro>
     <xacro:macro name="kinova_virtual_link" params="link_name">
@@ -85,10 +98,27 @@
         <child link="${child}"/>
         <axis xyz="${joint_axis_xyz}"/>
-        <limit effort="2000" velocity="1" lower="${joint_lower_limit}" upper="${joint_upper_limit}"/>
+        <limit effort="60" velocity="3.35" lower="${joint_lower_limit}" upper="${joint_upper_limit}"/>
         <origin xyz="${joint_origin_xyz}" rpy="${joint_origin_rpy}"/>
      </joint>
     </xacro:macro>
     <xacro:macro name="kinova_finger" params="prefix finger_number hand finger_origin_xyz finger_origin_rpy">
-        <xacro:kinova_armlink link_name="${prefix}link_finger_${finger_number}" link_mesh="finger_proximal" mesh_no="57"/>
+        <link name="${prefix}link_finger_${finger_number}">
+              <visual>
+                  <geometry>
+                      <mesh
+                          filename="package://kinova_description/meshes/finger_proximal.dae"/>
+                  </geometry>
+              </visual>
+              <collision>
+                  <geometry>
+                      <mesh
+                          filename="package://kinova_description/meshes/finger_proximal.dae"/>
+                  </geometry>
+              </collision>
+              <xacro:kinova_inertial mesh_no="1"/>
+        </link>
+        <gazebo reference="${prefix}link_finger_${finger_number}">
+            <material>Gazebo/Grey</material>
+        </gazebo>
         <joint name="${prefix}joint_finger_${finger_number}" type="revolute">
             <parent link="${hand}"/>
@@ -96,24 +126,44 @@
             <axis xyz="0 0 1"/>
             <origin xyz="${finger_origin_xyz}" rpy="${finger_origin_rpy}"/>
-            <limit lower="0" upper="2" effort="2000" velocity="1"/>
+            <limit lower="0" upper="2" effort="30" velocity="5"/>
+            <dynamics damping="0.7" friction="0.0"/>
         </joint>
-		    <transmission name="${prefix}joint_finger_${finger_number}_trans">
-					<type>transmission_interface/SimpleTransmission</type>
-					<joint name="${prefix}joint_finger_${finger_number}">
-					  <hardwareInterface>EffortJointInterface</hardwareInterface>
-					</joint>
-					<actuator name="${prefix}joint_finger_${finger_number}_actuator">
-					<hardwareInterface>EffortJointInterface</hardwareInterface>
-					<mechanicalReduction>1</mechanicalReduction>
-					</actuator>
-		    </transmission>
-        <xacro:kinova_armlink link_name="${prefix}link_finger_tip_${finger_number}" link_mesh="finger_distal" mesh_no="58"/>
-        <joint name="${prefix}joint_finger_tip_${finger_number}" type="fixed">
-            <parent link="${prefix}link_finger_${finger_number}"/>
-            <child link="${prefix}link_finger_tip_${finger_number}"/>
-            <axis xyz="0 0 1"/>
-            <origin xyz="0.044 -0.003 0" rpy="0 0 0"/>
-            <limit lower="0" upper="2" effort="2000" velocity="1"/>
-        </joint>
+        <transmission name="${prefix}joint_finger_${finger_number}_trans">
+          <type>transmission_interface/SimpleTransmission</type>
+          <joint name="${prefix}joint_finger_${finger_number}">
+            <hardwareInterface>EffortJointInterface</hardwareInterface>
+          </joint>
+          <actuator name="${prefix}joint_finger_${finger_number}_actuator">
+          <hardwareInterface>EffortJointInterface</hardwareInterface>
+          <mechanicalReduction>1</mechanicalReduction>
+          </actuator>
+        </transmission>
+        <link name="${prefix}link_finger_tip_${finger_number}">
+            <visual>
+                <geometry>
+                    <mesh
+                        filename="package://kinova_description/meshes/finger_distal.dae"/>
+                </geometry>
+            </visual>
+            <collision>
+                <geometry>
+                    <mesh
+                        filename="package://kinova_description/meshes/finger_distal.dae"/>
+                </geometry>
+            </collision>
+            <xacro:kinova_inertial mesh_no="58"/>
+      </link>
+      <gazebo reference="${prefix}link_finger_tip_${finger_number}">
+          <material>Gazebo/Grey</material>
+      </gazebo>
+      <joint name="${prefix}joint_finger_tip_${finger_number}" type="revolute">
+          <parent link="${prefix}link_finger_${finger_number}"/>
+          <child link="${prefix}link_finger_tip_${finger_number}"/>
+          <axis xyz="0 0 1"/>
+          <origin xyz="0.044 -0.003 0" rpy="0 0 0.3"/>
+          <limit lower="0" upper="2" effort="30" velocity="5"/>
+          <dynamics damping="0.0" friction="0.0"/>
+          <mimic joint="${prefix}joint_finger_${finger_number}" multiplier="0.6" offset="0.0"/>
+      </joint>
     </xacro:macro>
 </root>

File: kinova_description/urdf/kinova_inertial.xacro (robot description, xacro)
@@ -2,29 +2,29 @@
 <root xmlns:xi="http://www.w3.org/2001/XInclude"
 	xmlns:gazebo="http://playerstage.sourceforge.net/gazebo/xmlschema/#gz"
-    xmlns:model="http://playerstage.sourceforge.net/gazebo/xmlschema/#model"
+	xmlns:model="http://playerstage.sourceforge.net/gazebo/xmlschema/#model"
 	xmlns:sensor="http://playerstage.sourceforge.net/gazebo/xmlschema/#sensor"
 	xmlns:body="http://playerstage.sourceforge.net/gazebo/xmlschema/#body"
-    xmlns:geom="http://playerstage.sourceforge.net/gazebo/xmlschema/#geom"
-    xmlns:joint="http://playerstage.sourceforge.net/gazebo/xmlschema/#joint"
+	xmlns:geom="http://playerstage.sourceforge.net/gazebo/xmlschema/#geom"
+	xmlns:joint="http://playerstage.sourceforge.net/gazebo/xmlschema/#joint"
 	xmlns:controller="http://playerstage.sourceforge.net/gazebo/xmlschema/#controller"
 	xmlns:interface="http://playerstage.sourceforge.net/gazebo/xmlschema/#interface"
 	xmlns:rendering="http://playerstage.sourceforge.net/gazebo/xmlschema/#rendering"
-    xmlns:renderable="http://playerstage.sourceforge.net/gazebo/xmlschema/#renderable"
-    xmlns:physics="http://playerstage.sourceforge.net/gazebo/xmlschema/#physics"
+	xmlns:renderable="http://playerstage.sourceforge.net/gazebo/xmlschema/#renderable"
+	xmlns:physics="http://playerstage.sourceforge.net/gazebo/xmlschema/#physics"
 	xmlns:xacro="http://ros.org/wiki/xacro">
-<!-- links      		mesh_no
-   base           		0
-   shoulder       		1
-   arm            		2
-   forearm        		3
-   wrist          		4
-   arm_mico       		5
-   arm_half1 (7dof)		6
-   arm_half2 (7dof)		7
+<!-- links          mesh_no
+   base               0
+   shoulder           1
+   arm                2
+   forearm            3
+   wrist              4
+   arm_mico           5
+   arm_half1 (7dof)   6
+   arm_half2 (7dof)   7
    wrist_spherical_1  8
    wrist_spherical_2  9
-   hand 3 finger  		55
-   hand_2finger   		56
-   finger_proximal		57
+   hand 3 finger      55
+   hand_2finger       56
+   finger_proximal    57
    finger_distal      58
 -->

File: kinova_description/urdf/m1n6s200.xacro (robot description, xacro)
@@ -90,23 +90,23 @@
     <xacro:property name="joint_end_effector_origin_xyz" value="0 0 -0.1600" />
     <xacro:property name="joint_end_effector_origin_rpy" value="${J_PI} 0 0" />
-    <xacro:macro name="m1n6s200" params="base_parent prefix:=m1n6s200">
+    <xacro:macro name="m1n6s200" params="base_parent use_ring_mesh:=true prefix:=m1n6s200">
         <xacro:gazebo_config robot_namespace="${prefix}"/>
         <xacro:kinova_armlink link_name="${prefix}_link_base" link_mesh="${link_base_mesh}" mesh_no="${link_base_mesh_no}"/>
         <xacro:kinova_armjoint joint_name="${prefix}_joint_base" type="${joint_base_type}" parent="${base_parent}" child="${prefix}_link_base" joint_axis_xyz="${joint_base_axis_xyz}" joint_origin_xyz="${joint_base_origin_xyz}" joint_origin_rpy="${joint_base_origin_rpy}" joint_lower_limit="0" joint_upper_limit="0" fixed="true"/>
-        <xacro:kinova_armlink link_name="${prefix}_link_1" link_mesh="${link_1_mesh}" use_ring_mesh="true" mesh_no="${link_1_mesh_no}"/>
+        <xacro:kinova_armlink link_name="${prefix}_link_1" link_mesh="${link_1_mesh}" use_ring_mesh="${use_ring_mesh}" mesh_no="${link_1_mesh_no}"/>
         <xacro:kinova_armjoint joint_name="${prefix}_joint_1" type="${joint_1_type}" parent="${prefix}_link_base" child="${prefix}_link_1" joint_axis_xyz="${joint_1_axis_xyz}" joint_origin_xyz="${joint_1_origin_xyz}" joint_origin_rpy="${joint_1_origin_rpy}" joint_lower_limit="${joint_1_lower_limit}" joint_upper_limit="${joint_1_upper_limit}"/>
-        <xacro:kinova_armlink link_name="${prefix}_link_2" link_mesh="${link_2_mesh}" use_ring_mesh="true" mesh_no="${link_2_mesh_no}"/>
+        <xacro:kinova_armlink link_name="${prefix}_link_2" link_mesh="${link_2_mesh}" use_ring_mesh="${use_ring_mesh}" mesh_no="${link_2_mesh_no}"/>
         <xacro:kinova_armjoint joint_name="${prefix}_joint_2" type="${joint_2_type}" parent="${prefix}_link_1" child="${prefix}_link_2" joint_axis_xyz="${joint_2_axis_xyz}" joint_origin_xyz="${joint_2_origin_xyz}" joint_origin_rpy="${joint_2_origin_rpy}" joint_lower_limit="${joint_2_lower_limit}" joint_upper_limit="${joint_2_upper_limit}"/>
-        <xacro:kinova_armlink link_name="${prefix}_link_3" link_mesh="${link_3_mesh}" use_ring_mesh="true" mesh_no="${link_3_mesh_no}"/>
+        <xacro:kinova_armlink link_name="${prefix}_link_3" link_mesh="${link_3_mesh}" use_ring_mesh="${use_ring_mesh}" mesh_no="${link_3_mesh_no}"/>
         <xacro:kinova_armjoint joint_name="${prefix}_joint_3" type="${joint_3_type}" parent="${prefix}_link_2" child="${prefix}_link_3" joint_axis_xyz="${joint_3_axis_xyz}" joint_origin_xyz="${joint_3_origin_xyz}" joint_origin_rpy="${joint_3_origin_rpy}" joint_lower_limit="${joint_3_lower_limit}" joint_upper_limit="${joint_3_upper_limit}"/>
-        <xacro:kinova_armlink link_name="${prefix}_link_4" link_mesh="${link_4_mesh}" use_ring_mesh="true" ring_mesh="ring_small" mesh_no="${link_4_mesh_no}"/>
+        <xacro:kinova_armlink link_name="${prefix}_link_4" link_mesh="${link_4_mesh}" use_ring_mesh="${use_ring_mesh}" ring_mesh="ring_small" mesh_no="${link_4_mesh_no}"/>
         <xacro:kinova_armjoint joint_name="${prefix}_joint_4" type="${joint_4_type}" parent="${prefix}_link_3" child="${prefix}_link_4" joint_axis_xyz="${joint_4_axis_xyz}" joint_origin_xyz="${joint_4_origin_xyz}" joint_origin_rpy="${joint_4_origin_rpy}" joint_lower_limit="${joint_4_lower_limit}" joint_upper_limit="${joint_4_upper_limit}"/>
-        <xacro:kinova_armlink link_name="${prefix}_link_5" link_mesh="${link_5_mesh}" use_ring_mesh="true" ring_mesh="ring_small" mesh_no="${link_5_mesh_no}"/>
+        <xacro:kinova_armlink link_name="${prefix}_link_5" link_mesh="${link_5_mesh}" use_ring_mesh="${use_ring_mesh}" ring_mesh="ring_small" mesh_no="${link_5_mesh_no}"/>
         <xacro:kinova_armjoint joint_name="${prefix}_joint_5" type="${joint_5_type}" parent="${prefix}_link_4" child="${prefix}_link_5" joint_axis_xyz="${joint_5_axis_xyz}" joint_origin_xyz="${joint_5_origin_xyz}" joint_origin_rpy="${joint_5_origin_rpy}" joint_lower_limit="${joint_5_lower_limit}" joint_upper_limit="${joint_5_upper_limit}"/>
-        <xacro:kinova_armlink link_name="${prefix}_link_6" link_mesh="${link_6_mesh}" use_ring_mesh="true" ring_mesh="ring_small" mesh_no="${link_6_mesh_no}"/>
+        <xacro:kinova_armlink link_name="${prefix}_link_6" link_mesh="${link_6_mesh}" use_ring_mesh="${use_ring_mesh}" ring_mesh="ring_small" mesh_no="${link_6_mesh_no}"/>
         <xacro:kinova_armjoint joint_name="${prefix}_joint_6" type="${joint_6_type}" parent="${prefix}_link_5" child="${prefix}_link_6" joint_axis_xyz="${joint_6_axis_xyz}" joint_origin_xyz="${joint_6_origin_xyz}" joint_origin_rpy="${joint_6_origin_rpy}" joint_lower_limit="${joint_6_lower_limit}" joint_upper_limit="${joint_6_upper_limit}"/>
         <xacro:kinova_virtual_link link_name="${prefix}_end_effector"/>
         <xacro:kinova_virtual_joint joint_name="${prefix}_joint_end_effector" type="${joint_end_effector_type}" parent="${prefix}_link_6" child="${prefix}_end_effector" joint_axis_xyz="${joint_end_effector_axis_xyz}" joint_origin_xyz="${joint_end_effector_origin_xyz}" joint_origin_rpy="${joint_end_effector_origin_rpy}" joint_lower_limit="0" joint_upper_limit="0"/>
-    <xacro:kinova_2fingers link_hand="${prefix}_link_6" prefix="${prefix}_"/>
+        <xacro:kinova_2fingers link_hand="${prefix}_link_6" prefix="${prefix}_"/>
     </xacro:macro>
 </root>

File: kinova_description/urdf/m1n6s200_standalone.xacro (robot description, xacro)
@@ -23,10 +23,10 @@
     <!--<material name="Black" /> -->
     </visual>
-    <collision>
+    <!--collision>
       <origin xyz="0 0 0" rpy="0 0 0" />
       <geometry>
         <box size = "0.01 0.01 0.01"/>
       </geometry>
-    </collision>
+    </collision-->
   </link>
   <!-- for gazebo -->

File: kinova_description/urdf/two_arm_robot_example_standalone.xacro (robot description, xacro)
@@ -22,10 +22,10 @@
       </geometry>
     </visual>
-    <collision>
+    <!--collision>
       <origin xyz="0 0 0" rpy="0 0 0" />
       <geometry>
         <box size = "0.01 0.01 0.01"/>
       </geometry>
-    </collision>
+    </collision-->
   </link>
 	<link name="left_arm_mount">
